Commit message: Tranformation matrix is now calculated from current robot transform

File: urdf/gantry_ur5_z_full_movement.urdf.xacro (robot description, xacro)
@@ -10,6 +10,6 @@
   <xacro:property name="gantry_thickness" value="0.2"/>
   <xacro:property name="collision_offset" value="0.005"/>
-  <xacro:property name="movement_restriction_x" value="0.0"/>
-  <xacro:property name="movement_restriction_y" value="0.0"/>
+  <xacro:property name="movement_restriction_x" value="0.5"/>
+  <xacro:property name="movement_restriction_y" value="0.5"/>
   <xacro:macro name="piller" params="num x y">
 	<link name="gantry_piller_${num}">
